File: Hardware/0. Project/ChristmasTree.brd (EAGLE design)
At the start: 66.8 x 98.6 mm, 28 parts, among them CN1 CELL, CN2 Micro USB Type B, IC1 ATMEGA32U4-MU, U1 RT9193-33GB, Y1 8MHz

Commit message: WIP
Parts:
- removed C14: 1uF, microbuilder:0603-NO
- removed C9: 10uF, microbuilder:0805-NO
- removed IC1: ATMEGA32U4-MU, microbuilder:TQFN44_7MM
- added C2, C8: 1uF, My-RLC:C0603
- added C3, C4, C5, C7: 100nF, My-RLC:C0603
- added C6: 10uF, My-RLC:C0805
- added R9: 10k (5%), My-RLC:R0603
- added U3: ATMEGA32U4, SparkFun_Pro_Micro_v13a:TESTING_QFN-44
- R4, R5: value 22R -> 22R (5%)
- Y1: device SparkFun:RESONATOR-SMD -> crystal2:HC49UP
- moved Y1 167.7 mm to (-56.0, -238.6)
Connections:
- removed net +3V3: C9.1, IC1.14, IC1.24, IC1.33, IC1.34, IC1.44, IC1.6
- removed net A0: IC1.36
- removed net A1: IC1.37
- removed net A2: IC1.38
- removed net A3: IC1.39
- removed net A4: IC1.40
- removed net A5: IC1.41
- removed net AREF: C14.1, IC1.42
- removed net D0: IC1.20
- removed net D1: IC1.21
- removed net D10: IC1.30
- removed net D11: IC1.12
- removed net D12: IC1.26
- removed net D13: IC1.32
- removed net D4: IC1.25
- removed net D5: IC1.31
- removed net D6: IC1.27
- removed net D7: IC1.1
- removed net D8: IC1.28
- removed net D9: IC1.29
- removed net GND: C14.2, C9.2, IC1.15, IC1.23, IC1.35, IC1.43, IC1.5, Y1.2
- removed net MISO: IC1.11
- removed net MOSI: IC1.10
- removed net RST: IC1.13
- removed net SCK: IC1.9
- removed net SCL: IC1.18
- removed net SDA: IC1.19
- new net N$18: C7.1, U3.42
- new net N$19: U3.27
- new net P$1: U3.2, U3.7
- new net RESET: R9.1, U3.13
- net 0V: now also C2.2, C3.2, C4.2, C5.2, C6.2, C7.2, C8.2, U3.15, U3.23, U3.33, U3.35, U3.43, U3.5
- net 3.3V: now also C5.1, C8.1, R9.2, U3.14, U3.24, U3.34, U3.44
- net N$15: now also C3.1, U3.17, Y1.1; no longer IC1.16, Y1.3
- net N$16: now also C4.1, U3.16, Y1.2; no longer IC1.17, Y1.1
- net N$17: now also C2.1, U3.6; no longer CN2.1, D3.A
- net USB_D+: now also U3.4; no longer IC1.4
- net USB_D-: now also U3.3; no longer IC1.3
- net VBUS: now also C6.1, CN2.1, D3.A; no longer IC1.7

Commit message: PCB 100mm
Parts:
- removed U3: ATMEGA32U4, SparkFun_Pro_Micro_v13a:TESTING_QFN-44
- added LDR1: (no value), photo-elements:T0-46-A10XX
- added R3: 22R (5%), My-RLC:R0603
- added U2: ATMEGA32U4, SparkFun_Pro_Micro_v13a:TESTING_QFN-44
- C1: value 22nF -> 10uF; device My-RLC:C0603 -> My-RLC:C0805
- C2: value 1uF -> 22nF
- C3, C5: value 100nF -> 1uF
- C6: value 10uF -> 100nF; device My-RLC:C0805 -> My-RLC:C0603
- C8: value 1uF -> 100nF
- CN1: value CELL -> Micro USB Type B; device My-Battery:18650 -> My-Connectors:10118193-0001LF
- CN2: value Micro USB Type B -> CELL; device My-Connectors:10118193-0001LF -> My-Battery:18650
- R2: value 470R -> 22R (5%); device rcl:R0603 -> My-RLC:R0603
- R4: value 22R (5%) -> 470R; device My-RLC:R0603 -> rcl:R0603
- R5: value 22R (5%) -> 10k (5%)
- moved CN2 193.9 mm to (33.3, 32.8), turned to 90 degrees
- moved R2 178.1 mm to (-35.1, -160.8)
- moved R4 178.1 mm to (-17.8, 16.5)
- moved C2 119.4 mm to (-28.2, -108.4)
- moved R5 116.8 mm to (-98.0, -262.4)
- moved C1 84.0 mm to (-50.7, -189.3)
- moved CN1 42.0 mm to (-29.4, -150.8)
- moved C6 34.2 mm to (-56.3, -223.0)
- moved C5 24.8 mm to (-61.6, -223.0)
- moved LED2 20.3 mm to (-17.8, 10.2)
- moved LED4 20.3 mm to (-17.8, -10.2)
- moved C7 20.0 mm to (-66.9, -240.0)
- moved C3 12.2 mm to (-72.2, -251.0)
- moved C8 11.0 mm to (-72.2, -240.0)
- moved LED1 7.62 mm to (-17.8, 3.81)
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- renumbered D3 to D1, R9 to R1
Connections:
- removed net N$20: CN2.2, R4.1
- removed net N$23: CN2.3, R5.1
- removed net N$24: CN1.4, D2.A, SJ1.1
- removed net P$1: U3.2, U3.7
- new net LEDS_CONTROL: LED1.4-DIN, R4.2
- new net LIGHT_SENSOR: LDR1.2, R5.2, U2.36
- net 0V: now also CN1.MP1, CN1.MP2, CN1.MP3, CN1.MP4, R5.1, U2.15, U2.23, U2.33, U2.35, U2.43, U2.5; no longer CN2.MP1, CN2.MP2, CN2.MP3, CN2.MP4, U3.15, U3.23, U3.33, U3.35, U3.43, U3.5
- net 3.3V: now also C3.1, C4.1, LDR1.1, U2.14, U2.24, U2.34, U2.44; no longer C5.1, C8.1, U3.14, U3.24, U3.34, U3.44
- net N$11: now also LED4.2-DOUT; no longer LED2.2-DOUT
- net N$15: now also C7.1, U2.17; no longer C3.1, U3.17
- net N$16: now also C8.1, U2.16; no longer C4.1, U3.16
- net N$17: now also C5.1, U2.6; no longer C2.1, U3.6
- net N$18: now also C6.1, U2.42; no longer C7.1, U3.42
- net N$19: now also CN2.4, D2.A, SJ1.1; no longer U3.27
- net N$21: now also C2.1; no longer C1.1
- net N$3: now also R4.1, U2.27; no longer LED3.4-DIN, R2.2
- net N$4: now also LED2.2-DOUT, LED3.4-DIN; no longer LED1.4-DIN, LED4.2-DOUT
- net RESET: now also U2.13; no longer U3.13
- net USB_D+: now also CN1.3, R3.1, R3.2, U2.4; no longer R5.2, U3.4
- net USB_D-: now also CN1.2, R2.1, R2.2, U2.3; no longer R4.2, U3.3
- net VBUS: now also C1.1, CN1.1, U2.2, U2.7; no longer C6.1, CN2.1

Commit message: WIP
Parts:
- removed LED14: WS2812B, My-LED:5050
- added TP1, TP2: TPSQTP20R, testpad:TP20R
- CN2: value CELL -> 3.7V; device My-Battery:18650 -> My-Battery:JST-PH2
- moved R5 269.8 mm to (56.8, -41.5)
- moved C3 240.1 mm to (48.4, -43.4)
- moved C4 240.1 mm to (48.4, -37.9)
- moved C5 240.1 mm to (59.0, -15.4)
- moved C6 240.1 mm to (64.3, -15.4)
- moved C7 240.1 mm to (53.7, -32.4)
- moved C8 240.1 mm to (48.4, -32.4)
- moved R1 240.1 mm to (69.6, -16.7)
- moved Y1 240.1 mm to (64.6, -31.0)
- moved LED13 193.6 mm to (50.9, 135.9)
- moved C1 179.0 mm to (40.5, -35.2)
- moved CN1 175.6 mm to (51.5, 5.11), flipped to the bottom, turned to 90 degrees
- moved LED12 173.2 mm to (41.8, 114.4)
- moved LED11 163.3 mm to (55.8, 108.0)
- moved R2 145.2 mm to (36.4, -34.4)
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Connections:
- removed net N$12: LED13.2-DOUT, LED14.4-DIN
- net 0V: now also CN2.2; no longer CN2.5, LED14.3-GND
- net 3.3V: no longer LED14.1-VDD
- net N$19: now also CN2.1; no longer CN2.4
Other:
- board size 66.8 x 98.6 mm -> 99.3 x 147.7 mm

Commit message: PCB 1.0 done
Parts:
- added C10, C11, C12, C13, C14, C15, C16, C17, C18, C19, C20, C21, C9: 100nF, My-RLC:C0603
- LDR1: value (none) -> A1050_09
- R4: device rcl:R0603 -> My-RLC:R0603
- Y1: device crystal2:HC49UP -> crystal-geyer_V1_0:5.0X3.2_KX-9A
- moved R3 55.6 mm to (55.1, 14.7), flipped to the bottom, turned to 270 degrees
- moved R2 52.0 mm to (53.5, 14.7), flipped to the bottom, turned to 270 degrees
- moved R5 46.8 mm to (48.6, 4.64), flipped to the bottom, turned to 180 degrees
- moved C3 46.4 mm to (48.6, 3.04), flipped to the bottom
- moved C8 45.0 mm to (69.0, 7.60), flipped to the bottom, turned to 270 degrees
- moved R4 44.3 mm to (56.0, 2.88), flipped to the bottom, turned to 0 degrees
- moved C4 43.5 mm to (62.6, 3.24), flipped to the bottom, turned to 180 degrees
- moved C1 40.5 mm to (33.9, 4.76), flipped to the bottom, turned to 270 degrees
- moved Y1 37.3 mm to (66.3, 6.32), flipped to the bottom, turned to 90 degrees
- moved C7 37.2 mm to (65.9, 2.72), flipped to the bottom, turned to 180 degrees
- moved C2 36.6 mm to (48.5, 6.19), flipped to the bottom
- moved C6 32.6 mm to (51.8, 14.7), flipped to the bottom, turned to 90 degrees
- moved C5 30.2 mm to (56.6, 14.7), flipped to the bottom, turned to 90 degrees
- moved D2 30.0 mm to (43.1, 7.05), flipped to the bottom, turned to 270 degrees
- moved SJ1 28.9 mm to (42.8, 2.54), flipped to the bottom
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- renumbered TP1 to MH1, TP2 to MH2
Connections:
- new net N$12: R3.2, U2.4
- new net N$20: R2.2, U2.3
- net 0V: now also C10.2, C11.2, C12.2, C13.2, C14.2, C15.2, C16.2, C17.2, C18.2, C19.2, C20.2, C21.2, C9.2
- net 3.3V: now also C10.1, C11.1, C12.1, C13.1, C14.1, C15.1, C16.1, C17.1, C18.1, C19.1, C20.1, C21.1, C9.1
- net N$16: now also Y1.3; no longer Y1.2
- net USB_D+: no longer R3.2, U2.4
- net USB_D-: no longer R2.2, U2.3
Routing:
- net 3.3V: track 0.00 -> 527.7 mm, vias 0 -> 17
- net 0V: track 0.00 -> 454.9 mm, vias 0 -> 73
- net LEDS_CONTROL: track 0.00 -> 55.0 mm, vias 0 -> 3
- net N$11: track 0.00 -> 51.2 mm, vias 0 -> 2
- net N$4: track 0.00 -> 47.6 mm, vias 0 -> 2
- net N$9: track 0.00 -> 40.8 mm, vias 0 -> 2
- net N$1: track 0.00 -> 38.6 mm, vias 0 -> 2
- net VBUS: track 0.00 -> 36.7 mm, vias 0 -> 3
- net N$7: track 0.00 -> 36.1 mm, vias 0 -> 2
- net USB_D+: track 0.00 -> 32.8 mm
- net USB_D-: track 0.00 -> 29.6 mm
- net LIGHT_SENSOR: track 0.00 -> 24.8 mm, vias 0 -> 2
- net N$8: track 0.00 -> 24.4 mm, vias 0 -> 2
- net N$2: track 0.00 -> 24.2 mm, vias 0 -> 2
- net N$10: track 0.00 -> 23.7 mm, vias 0 -> 2
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- added copper zone on layer 1, net 0V
- added copper zone on layer 16, net 0V
Other:
- board text added: "2020 Coronavirus Pandemic Quarantine Projects"
- board text added: "Tiago Silva"

Commit message: Basic firmware test
Parts:
- LDR1: value A1050_09 -> (none)
- R5: value 10k (5%) -> 100k (5%)
Changed lines of the file:
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@@
 <drawing>
 <settings>
-<setting alwaysvectorfont="yes"/>
+<setting alwaysvectorfont="no"/>
 <setting verticaltext="up"/>
 </settings>
-<grid distance="2" unitdist="mil" unit="mil" style="lines" multiple="1" display="yes" altdistance="0.00127" altunitdist="mm" altunit="mm"/>
+<grid distance="1" unitdist="mil" unit="mil" style="lines" multiple="1" display="yes" altdistance="0.00127" altunitdist="mm" altunit="mm"/>
 <layers>
 <layer number="1" name="Top" color="4" fill="1" visible="yes" active="yes"/>
@@
 </layers>
 <board>
-<fusionsync huburn="a.cGVyc29uYWw6dWUyOTAyNzk3" projecturn="a.cGVyc29uYWw6dWUyOTAyNzk3IzIwMjAwOTI0MzM2MzczOTUx" f3durn="urn:adsk.wipprod:dm.lineage:wMaRPNqrQ3yQGWGDxtz49w" pcbguid="58c5647e-bc3e-46ae-93d2-734a1404439c" lastpulledtime="" lastsyncedchangeguid="" latestrevisionid="20f0e67f-7d68-4a19-83e3-bd85bdef268f" lastsyncedrevisionid="20f0e67f-7d68-4a19-83e3-bd85bdef268f" lastboardhashguid="aacab1c3-18f1-8c59-b34c-718e414a3054" lastpushedtime="2020-09-27T17:47:06Z" linktopcb3d="true"/>
+<fusionsync huburn="a.cGVyc29uYWw6dWUyOTAyNzk3" projecturn="a.cGVyc29uYWw6dWUyOTAyNzk3IzIwMjAwOTI0MzM2MzczOTUx" f3durn="urn:adsk.wipprod:dm.lineage:wMaRPNqrQ3yQGWGDxtz49w" pcbguid="" lastpulledtime="" lastsyncedchangeguid="" latestrevisionid="20f0e67f-7d68-4a19-83e3-bd85bdef268f" lastsyncedrevisionid="20f0e67f-7d68-4a19-83e3-bd85bdef268f" lastboardhashguid="aacab1c3-18f1-8c59-b34c-718e414a3054" lastpushedtime="2020-09-27T17:47:06Z" linktopcb3d="true"/>
 <plain>
 <wire x1="13.35336875" y1="1.095690625" x2="13.46946875" y2="1.502040625" width="0.000459375" layer="20" locked="yes"/>
@@
 <element name="C3" library="My-RLC" package="C0603" package3d_urn="urn:adsk.eagle:package:23494015/2" value="1uF" x="48.578" y="3.037" smashed="yes" rot="MR0">
 <attribute name="NAME" x="50.904" y="3.044" size="0.8128" layer="26" font="vector" ratio="15" rot="MR180" align="center"/>
+<attribute name="SPICEPREFIX" value="C" x="48.578" y="3.037" size="1.778" layer="28" rot="MR0" display="off"/>
 <attribute name="VALUE" x="48.832" y="0.243" size="0.6096" layer="28" ratio="10" rot="MR0" display="off"/>
 </element>
-<element name="LDR1" library="photo-elements" package="T0-46-A10XX" package3d_urn="urn:adsk.eagle:package:23501050/2" override_package3d_urn="urn:adsk.eagle:package:23536266/2" override_package_urn="urn:adsk.eagle:footprint:23536267/1" value="A1050_09" x="51.216" y="20.006" smashed="yes" rot="MR270">
+<element name="LDR1" library="photo-elements" package="T0-46-A10XX" package3d_urn="urn:adsk.eagle:package:23501050/2" override_package3d_urn="urn:adsk.eagle:package:23536266/2" override_package_urn="urn:adsk.eagle:footprint:23536267/1" value="" x="51.216" y="20.006" smashed="yes" rot="MR270">
 <attribute name="NAME" x="56.296" y="20.661" size="1.27" layer="26" rot="MR270" display="off"/>
 <attribute name="POPULARITY" value="0" x="51.216" y="20.006" size="1.778" layer="28" rot="MR270" display="off"/>
 <attribute name="VALUE" x="47.406" y="21.911" size="1.27" layer="28" rot="MR270" display="off"/>
 </element>
-<element name="R5" library="My-RLC" package="R0603" package3d_urn="urn:adsk.eagle:package:23494030/2" value="10k (5%)" x="48.561" y="4.645" smashed="yes" rot="MR180">
+<element name="R5" library="My-RLC" package="R0603" package3d_urn="urn:adsk.eagle:package:23494030/2" value="100k (5%)" x="48.561" y="4.645" smashed="yes" rot="MR180">
 <attribute name="NAME" x="50.936" y="4.632" size="0.8128" layer="26" font="vector" ratio="15" rot="MR180" align="center"/>
 <attribute name="VALUE" x="47.037" y="6.169" size="0.6096" layer="28" ratio="10" rot="MR180" display="off"/>

Commit message: Adequacy of values in some components
Parts:
- C2: value 22nF -> 10nF
- R4: value 470R -> 150R
- R5: value 100k (5%) -> 220k (5%)
- Y1: value 8MHz -> 16MHz
Changed lines of the file:
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@@
 <attribute name="NAME" x="48.0375" y="31.3395" size="0.8128" layer="25" ratio="10" rot="R270" display="off"/>
 </element>
-<element name="R4" library="My-RLC" package="R0603" package3d_urn="urn:adsk.eagle:package:23494030/2" value="470R" x="56.041" y="2.875" smashed="yes" rot="MR0">
+<element name="R4" library="My-RLC" package="R0603" package3d_urn="urn:adsk.eagle:package:23494030/2" value="150R" x="56.041" y="2.875" smashed="yes" rot="MR0">
 <attribute name="NAME" x="54" y="2.844" size="0.8128" layer="26" font="vector" ratio="15" rot="MR270" align="center"/>
 <attribute name="VALUE" x="56.676" y="0.97" size="1.27" layer="28" rot="MR0" display="off"/>
@@
 <attribute name="NAME" x="41.761" y="10.915" size="0.8128" layer="26" font="vector" ratio="15" rot="MR180" align="center"/>
 </element>
-<element name="C2" library="My-RLC" package="C0603" package3d_urn="urn:adsk.eagle:package:23494015/2" value="22nF" x="48.54" y="6.193" smashed="yes" rot="MR0">
+<element name="C2" library="My-RLC" package="C0603" package3d_urn="urn:adsk.eagle:package:23494015/2" value="10nF" x="48.54" y="6.193" smashed="yes" rot="MR0">
 <attribute name="NAME" x="50.935" y="6.169" size="0.8128" layer="26" font="vector" ratio="15" rot="MR0" align="center"/>
 <attribute name="VALUE" x="48.794" y="3.399" size="0.6096" layer="28" ratio="10" rot="MR0" display="off"/>
@@
 <attribute name="VALUE" x="53.844" y="14.475" size="0.6096" layer="28" ratio="10" rot="MR90" display="off"/>
 </element>
-<element name="Y1" library="crystal-geyer_V1_0" library_urn="urn:adsk.eagle:library:203" package="5.0X3.2_KX-9A" package3d_urn="urn:adsk.eagle:package:11927/1" override_package3d_urn="urn:adsk.eagle:package:23536242/2" override_package_urn="urn:adsk.eagle:footprint:11874/1" value="8MHz" x="66.271" y="6.322" smashed="yes" rot="MR90">
+<element name="Y1" library="crystal-geyer_V1_0" library_urn="urn:adsk.eagle:library:203" package="5.0X3.2_KX-9A" package3d_urn="urn:adsk.eagle:package:11927/1" override_package3d_urn="urn:adsk.eagle:package:23536242/2" override_package_urn="urn:adsk.eagle:footprint:11874/1" value="16MHz" x="66.271" y="6.322" smashed="yes" rot="MR90">
 <attribute name="NAME" x="68.715" y="6.355" size="0.8128" layer="26" font="vector" ratio="15" rot="MR0" align="center"/>
 <attribute name="VALUE" x="62.08" y="0.607" size="1.27" layer="28" ratio="10" rot="MR90" display="off"/>
@@
 <attribute name="VALUE" x="47.406" y="21.911" size="1.27" layer="28" rot="MR270" display="off"/>
 </element>
-<element name="R5" library="My-RLC" package="R0603" package3d_urn="urn:adsk.eagle:package:23494030/2" value="100k (5%)" x="48.561" y="4.645" smashed="yes" rot="MR180">
+<element name="R5" library="My-RLC" package="R0603" package3d_urn="urn:adsk.eagle:package:23494030/2" value="220k (5%)" x="48.561" y="4.645" smashed="yes" rot="MR180">
 <attribute name="NAME" x="50.936" y="4.632" size="0.8128" layer="26" font="vector" ratio="15" rot="MR180" align="center"/>
 <attribute name="VALUE" x="47.037" y="6.169" size="0.6096" layer="28" ratio="10" rot="MR180" display="off"/>
